File: VColChoc44.kicad_pcb (KiCad board)
At the start: 2 copper layers, 234 x 88 mm, 121 parts, among them J1 USB_C_Receptacle_USB2.0, SW1 SW_SPDT, SW2 SW_SPST, U1 CherryMX_LTST-A683CEGBW-Rotat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, U10 CherryMX_LTST-A683CEGBW-Rotat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, U11 CherryMX_LTST-A683CEGBW-Rotat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, U12 CherryMX_LTST-A683CEGBW-Rotat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, U13 CherryMX_LTST-A683CEGBW-Rotat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, U14 CherryMX_LTST-A683CEGBW-Rotat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, U15 CherryMX_LTST-A683CEGBW-Rotat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, U16 CherryMX_LTST-A683CEGBW-Rotat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, U17 CherryMX_LTST-A683CEGBW-Rotat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, U18 CherryMX_LTST-A683CEGBW-Rotat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, U19 CherryMX_LTST-A683CEGBW-Rotat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, U2 CherryMX_LTST-A683CEGBW-Rotat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, U20 CherryMX_LTST-A683CEGBW-Rotat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, U21 CherryMX_LTST-A683CEGBW-Rotat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, U22 CherryMX_LTST-A683CEGBW-Rotat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, U23 CherryMX_LTST-A683CEGBW-Rotat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, U24 CherryMX_LTST-A683CEGBW-Rotat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, U25 CherryMX_LTST-A683CEGBW-Rotat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, U26 CherryMX_LTST-A683CEGBW-Rotat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, U27 CherryMX_LTST-A683CEGBW-Rotat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, U28 CherryMX_LTST-A683CEGBW-Rotat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, U29 CherryMX_LTST-A683CEGBW-Rotat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, U3 CherryMX_LTST-A683CEGBW-Rotat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, U30 CherryMX_LTST-A683CEGBW-Rotat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, U31 CherryMX_LTST-A683CEGBW-Rotat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, U32 CherryMX_LTST-A683CEGBW-Rotat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, U33 CherryMX_LTST-A683CEGBW-Rotat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, U34 CherryMX_LTST-A683CEGBW-Rotat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, U35 CherryMX_LTST-A683CEGBW-Rotat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, U36 CherryMX_LTST-A683CEGBW-Rotat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, U37 CherryMX_LTST-A683CEGBW-Rotat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, U38 CherryMX_LTST-A683CEGBW-Rotat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, U39 CherryMX_LTST-A683CEGBW-Rotat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, U4 CherryMX_LTST-A683CEGBW-Rotat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, U40 CherryMX_LTST-A683CEGBW-Rotat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, U41 CherryMX_LTST-A683CEGBW-Rotat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, U42 CherryMX_LTST-A683CEGBW-Rotat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, U43 CherryMX_LTST-A683CEGBW-Rotat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, U44 CherryMX_LTST-A683CEGBW-Rotat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, U45 W25Q128JVS, U46 RP2040, U47 AMS1117-3.3, U5 CherryMX_LTST-A683CEGBW-Rotat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, U6 CherryMX_LTST-A683CEGBW-Rotat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, U7 CherryMX_LTST-A683CEGBW-Rotat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, U8 CherryMX_LTST-A683CEGBW-Rotat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, U9 CherryMX_LTST-A683CEGBW-Rotat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, Y1 12MHz

Commit message: initial
Parts:
- removed C10, C4, C5, C6, C7, C8, C9: 100n, Capacitor_SMD:C_0603_1608Metric
- removed C11, C12: 1u, Capacitor_SMD:C_0603_1608Metric
- removed C13, C16: 22p, Capacitor_SMD:C_0603_1608Metric
- removed C14, C15: 22u, Capacitor_SMD:C_0603_1608Metric
- removed D10, D11, D12, D13, D14, D15, D16, D17, D18, D19, D20, D21, D22, D23, D24, D25, D26, D27, D28, D29, D30, D31, D32, D33, D34, D35, D36, D37, D38, D39, D4, D40, D41, D42, D43, D44, D5, D6, D7, D8, D9: D, Diode_SMD:D_SOD-123
- removed D45: RED, LED_SMD:LED_0603_1608Metric
- removed R7, R8: 1k, Resistor_SMD:R_0603_1608Metric
- removed U47: AMS1117-3.3, Package_TO_SOT_SMD:SOT-223-3_TabPin2
- added H1: MountingHole, MountingHole:MountingHole_2.2mm_M2_DIN965, F.Cu at (55.0, 130.0)
- added H10: MountingHole, MountingHole:MountingHole_2.2mm_M2_DIN965, F.Cu at (150.0, 75.0)
- added H2: MountingHole, MountingHole:MountingHole_2.2mm_M2_DIN965, F.Cu at (105.0, 140.0)
- added H3: MountingHole, MountingHole:MountingHole_2.2mm_M2_DIN965, F.Cu at (195.0, 140.0)
- added H4: MountingHole, MountingHole:MountingHole_2.2mm_M2_DIN965, F.Cu at (245.0, 130.0)
- added H5: MountingHole, MountingHole:MountingHole_2.2mm_M2_DIN965, F.Cu at (150.0, 142.5)
- added H6: MountingHole, MountingHole:MountingHole_2.2mm_M2_DIN965, F.Cu at (65.0, 62.5)
- added H7: MountingHole, MountingHole:MountingHole_2.2mm_M2_DIN965, F.Cu at (235.0, 62.5)
- added H8: MountingHole, MountingHole:MountingHole_2.2mm_M2_DIN965, F.Cu at (120.0, 62.5)
- added H9: MountingHole, MountingHole:MountingHole_2.2mm_M2_DIN965, F.Cu at (180.0, 62.5)
- added J2: USB_C_Receptacle_USB2.0, Connector_USB:USB_C_Receptacle_HRO_TYPE-C-31-M-12, B.Cu at (150.0, 63.6)
- added J3: Conn_01x04, Connector_PinHeader_2.54mm:PinHeader_1x04_P2.54mm_Vertical, F.Cu at (155.0, 102.5)
- added L1: 10uH, Inductor_SMD:L_0805_2012Metric, B.Cu at (145.8, 91.0)
- C1, C2: value 100n -> 22pF
- C3: value 100n -> 10uF
- D1: value D -> KT-0603R; footprint Diode_SMD:D_SOD-123 -> LED_SMD:LED_0603_1608Metric
- D2: value D -> 19-217/BHC-ZL1M2RY/3T; footprint Diode_SMD:D_SOD-123 -> LED_SMD:LED_0603_1608Metric
- D3: value D -> 19-217/GHC-YR1S2/3T; footprint Diode_SMD:D_SOD-123 -> LED_SMD:LED_0603_1608Metric
- J1: value USB_C_Receptacle_USB2.0 -> Conn_01x02_Male; footprint Connector_USB:USB_C_Receptacle_HRO_TYPE-C-31-M-12 -> Connector_PinHeader_2.54mm:PinHeader_1x02_P2.54mm_Vertical
- R1, R2: value 5.1k -> 1K
- R3: value DNP -> 5k1
- R4: value 1k -> 5k1
- R5: value 22 -> 1K
- R6: value 22 -> 10K
- SW1: footprint Button_Switch_SMD:SW_SPDT_PCM12 -> E73:SPDT_C128955
- SW2: value SW_SPST -> SW_Push; footprint Button_Switch_SMD:SW_SPST_TL3342 -> E73:SW_TACT_ALPS_SKQGABE010
- U1, U10, U11, U12, U13, U14, U15, U16, U17, U18, U19, U2, U20, U21, U22, U23, U24, U25, U26, U27, U28, U29, U3, U30, U31, U32, U33, U34, U35, U36, U37, U38, U39, U4, U40, U41, U42, U43, U44, U5, U6, U7, U8, U9: value CherryMX_LTST-A683CEGBW-Rotated -> diode-choc; footprint keyswitches:Kailh_socket_PG1350_sk6812mini_e -> pg1232:pg1232-D
- U45: value W25Q128JVS -> E73-2G4M08S1C-52840; footprint Package_SO:SOIC-8_5.23x5.23mm_P1.27mm -> nrfmicro:E73-2G4M08S1C-52840
- U46: value RP2040 -> TP4054; footprint MCU_RaspberryPi_and_Boards:RP2040-QFN-56 -> Package_TO_SOT_SMD:TSOT-23-5
- Y1: value 12MHz -> 32,768; footprint Crystal:Crystal_SMD_3225-4Pin_3.2x2.5mm -> Crystal:Crystal_SMD_3215-2Pin_3.2x1.5mm
- moved D1 83.4 mm to (143.0, 62.0), turned to 90 degrees
- moved SW2 73.7 mm to (134.7, 63.4), turned to 180 degrees
- moved D2 63.0 mm to (141.2, 62.0), turned to 90 degrees
- moved LS1 60.5 mm to (150.0, 127.5), turned to 270 degrees
- moved D3 59.4 mm to (157.0, 62.0), turned to 90 degrees
- moved SW1 41.6 mm to (162.5, 62.5), turned to 180 degrees
- moved U46 23.4 mm to (166.2, 75.8), turned to 10 degrees
- moved R6 23.3 mm to (169.7, 75.0), turned to 280 degrees
- moved R4 22.7 mm to (142.2, 67.6), turned to 180 degrees
- moved U45 21.3 mm to (142.0, 93.0), turned to 260 degrees
- moved Y1 20.1 mm to (138.7, 88.8), turned to 170 degrees
- moved R5 19.6 mm to (157.0, 65.0)
- moved C1 18.3 mm to (135.4, 88.0), turned to 80 degrees
- moved J1 18.1 mm to (162.1, 77.5), turned to 10 degrees
- moved C2 12.8 mm to (141.9, 89.2), turned to 260 degrees
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Connections:
- C1 pad 1: +1V1 -> Net-(C1-Pad1)
- C2 pad 1: +1V1 -> GND
- C2 pad 2: GND -> Net-(C2-Pad2)
- C3 pad 1: +3V3 -> VBAT
- D1 pad 1: ROW1 -> Net-(D1-Pad1)
- D1 pad 2: Net-(D1-Pad2) -> RED_LED
- D2 pad 1: ROW1 -> Net-(D2-Pad1)
- D2 pad 2: Net-(D2-Pad2) -> BLUE_LED
- D3 pad 1: ROW1 -> Net-(D3-Pad1)
- D3 pad 2: Net-(D3-Pad2) -> VBUS
- R1 pad 1: GND -> Net-(D1-Pad1)
- R1 pad 2: Net-(J1-PadA5) -> GND
- R2 pad 1: GND -> Net-(D2-Pad1)
- R2 pad 2: Net-(J1-PadB5) -> GND
- R3 pad 1: /RP2040/QSPISS -> Net-(J2-PadB5)
- R3 pad 2: +3V3 -> GND
- R4 pad 1: /RP2040/QSPISS -> Net-(J2-PadA5)
- R4 pad 2: Net-(R4-Pad2) -> GND
- R5 pad 1: Data+ -> Net-(D3-Pad1)
- R6 pad 1: Data- -> GND
- SW1 pad 1: (no net) -> VBAT
- SW1 pad 2: GND -> Net-(J1-Pad1)
- SW1 pad 3: Net-(R4-Pad2) -> Net-(SW1-Pad3)
- SW2 pad 2: /RP2040/RESET -> RESET
- U1 pad 1: Net-(D1-Pad2) -> COL1
- U1 pad 2: COL1 -> ROW1
- U1 pad 3: GND -> (no net)
- U1 pad 4: RGBData1 -> (no net)
- U1 pad 5: RGB2 -> (no net)
- U10 pad 1: Net-(D10-Pad2) -> COL10
- U10 pad 2: COL10 -> ROW1
- U10 pad 3: GND -> (no net)
- U10 pad 4: RGB43 -> (no net)
- U10 pad 5: RGB44 -> (no net)
- U11 pad 1: Net-(D11-Pad2) -> COL11
- U11 pad 2: COL11 -> ROW1
- U11 pad 3: GND -> (no net)
- U11 pad 4: RGB44 -> (no net)
- U12 pad 1: Net-(D12-Pad2) -> COL1
- U12 pad 2: COL1 -> ROW2
- U12 pad 3: GND -> (no net)
- U12 pad 4: RGB6 -> (no net)
- U12 pad 5: RGB7 -> (no net)
- U13 pad 1: Net-(D13-Pad2) -> COL2
- U13 pad 2: COL2 -> ROW2
- U13 pad 3: GND -> (no net)
- U13 pad 4: RGB7 -> (no net)
- U13 pad 5: RGB8 -> (no net)
- U14 pad 1: Net-(D14-Pad2) -> COL3
- U14 pad 2: COL3 -> ROW2
- U14 pad 3: GND -> (no net)
- U14 pad 4: RGB8 -> (no net)
- U14 pad 5: RGB9 -> (no net)
- U15 pad 1: Net-(D15-Pad2) -> COL4
- U15 pad 2: COL4 -> ROW2
- U15 pad 3: GND -> (no net)
- U15 pad 4: RGB9 -> (no net)
- U15 pad 5: RGB10 -> (no net)
- U16 pad 1: Net-(D16-Pad2) -> COL5
- U16 pad 2: COL5 -> ROW2
- U16 pad 3: GND -> (no net)
- U16 pad 4: RGB10 -> (no net)
- U16 pad 5: RGB11 -> (no net)
- U17 pad 1: Net-(D17-Pad2) -> COL6
- U17 pad 2: COL6 -> ROW2
- U17 pad 3: GND -> (no net)
- U17 pad 4: RGB22 -> (no net)
- U17 pad 5: RGB23 -> (no net)
- U18 pad 1: Net-(D18-Pad2) -> COL7
- U18 pad 2: COL7 -> ROW2
- U18 pad 3: GND -> (no net)
- U18 pad 4: RGB35 -> (no net)
- U18 pad 5: RGB36 -> (no net)
- U19 pad 1: Net-(D19-Pad2) -> COL8
- U19 pad 2: COL8 -> ROW2
- U19 pad 3: GND -> (no net)
- U19 pad 4: RGB36 -> (no net)
- U19 pad 5: RGB37 -> (no net)
- U2 pad 1: Net-(D2-Pad2) -> COL2
- U2 pad 2: COL2 -> ROW1
- U2 pad 3: GND -> (no net)
- U2 pad 4: RGB2 -> (no net)
- U2 pad 5: RGB3 -> (no net)
- U20 pad 1: Net-(D20-Pad2) -> COL9
- U20 pad 2: COL9 -> ROW2
- U20 pad 3: GND -> (no net)
- U20 pad 4: RGB37 -> (no net)
- U20 pad 5: RGB38 -> (no net)
- U21 pad 1: Net-(D21-Pad2) -> COL10
- U21 pad 2: COL10 -> ROW2
- U21 pad 3: GND -> (no net)
- U21 pad 4: RGB38 -> (no net)
- U21 pad 5: RGB39 -> (no net)
- U22 pad 1: Net-(D22-Pad2) -> COL11
- U22 pad 2: COL11 -> ROW2
- U22 pad 3: GND -> (no net)
- U22 pad 4: RGB39 -> (no net)
- U22 pad 5: RGB40 -> (no net)
- U23 pad 1: Net-(D23-Pad2) -> COL1
- U23 pad 2: COL1 -> ROW3
- U23 pad 3: GND -> (no net)
- U23 pad 4: RGB11 -> (no net)
- U23 pad 5: RGB12 -> (no net)
- U24 pad 1: Net-(D24-Pad2) -> COL2
- U24 pad 2: COL2 -> ROW3
- U24 pad 3: GND -> (no net)
- U24 pad 4: RGB12 -> (no net)
- U24 pad 5: RGB13 -> (no net)
- U25 pad 1: Net-(D25-Pad2) -> COL3
- U25 pad 2: COL3 -> ROW3
- U25 pad 3: GND -> (no net)
- U25 pad 4: RGB13 -> (no net)
- U25 pad 5: RGB14 -> (no net)
- U26 pad 1: Net-(D26-Pad2) -> COL4
- U26 pad 2: COL4 -> ROW3
- U26 pad 3: GND -> (no net)
- U26 pad 4: RGB14 -> (no net)
- U26 pad 5: RGB15 -> (no net)
- U27 pad 1: Net-(D27-Pad2) -> COL5
- U27 pad 2: COL5 -> ROW3
- U27 pad 3: GND -> (no net)
- U27 pad 4: RGB15 -> (no net)
- U27 pad 5: RGB16 -> (no net)
- U28 pad 1: Net-(D28-Pad2) -> COL6
- U28 pad 2: COL6 -> ROW3
- U28 pad 3: GND -> (no net)
- U28 pad 4: RGB29 -> (no net)
- U28 pad 5: RGB30 -> (no net)
- U29 pad 1: Net-(D29-Pad2) -> COL7
- U29 pad 2: COL7 -> ROW3
- U29 pad 3: GND -> (no net)
- U29 pad 4: RGB30 -> (no net)
- U29 pad 5: RGB31 -> (no net)
- U3 pad 1: Net-(D3-Pad2) -> COL3
- U3 pad 2: COL3 -> ROW1
- U3 pad 3: GND -> (no net)
- U3 pad 4: RGB3 -> (no net)
- U3 pad 5: RGB4 -> (no net)
- U30 pad 1: Net-(D30-Pad2) -> COL8
- U30 pad 2: COL8 -> ROW3
- U30 pad 3: GND -> (no net)
- U30 pad 4: RGB31 -> (no net)
- U30 pad 5: RGB32 -> (no net)
- U31 pad 1: Net-(D31-Pad2) -> COL9
- U31 pad 2: COL9 -> ROW3
- U31 pad 3: GND -> (no net)
- U31 pad 4: RGB32 -> (no net)
- U31 pad 5: RGB33 -> (no net)
- U32 pad 1: Net-(D32-Pad2) -> COL10
- U32 pad 2: COL10 -> ROW3
- U32 pad 3: GND -> (no net)
- U32 pad 4: RGB33 -> (no net)
- U32 pad 5: RGB34 -> (no net)
- U33 pad 1: Net-(D33-Pad2) -> COL11
- U33 pad 2: COL11 -> ROW3
- U33 pad 3: GND -> (no net)
- U33 pad 4: RGB34 -> (no net)
- U33 pad 5: RGB35 -> (no net)
- U34 pad 1: Net-(D34-Pad2) -> COL1
- U34 pad 2: COL1 -> ROW4
- U34 pad 3: GND -> (no net)
- U34 pad 4: RGB17 -> (no net)
- U34 pad 5: RGB18 -> (no net)
- U35 pad 1: Net-(D35-Pad2) -> COL2
- U35 pad 2: COL2 -> ROW4
- U35 pad 3: GND -> (no net)
- U35 pad 4: RGB18 -> (no net)
- U35 pad 5: RGB19 -> (no net)
- U36 pad 1: Net-(D36-Pad2) -> COL3
- U36 pad 2: COL3 -> ROW4
- U36 pad 3: GND -> (no net)
- U36 pad 4: RGB19 -> (no net)
- U36 pad 5: RGB20 -> (no net)
- U37 pad 1: Net-(D37-Pad2) -> COL4
- U37 pad 2: COL4 -> ROW4
- U37 pad 3: GND -> (no net)
- U37 pad 4: RGB20 -> (no net)
- U37 pad 5: RGB21 -> (no net)
- U38 pad 1: Net-(D38-Pad2) -> COL5
- U38 pad 2: COL5 -> ROW4
- U38 pad 3: GND -> (no net)
- U38 pad 4: RGB21 -> (no net)
- U38 pad 5: RGB22 -> (no net)
- U39 pad 1: Net-(D39-Pad2) -> COL6
- U39 pad 2: COL6 -> ROW4
- U39 pad 3: GND -> (no net)
- U39 pad 4: RGB23 -> (no net)
- U39 pad 5: RGB24 -> (no net)
- U4 pad 1: Net-(D4-Pad2) -> COL4
- U4 pad 2: COL4 -> ROW1
- U4 pad 3: GND -> (no net)
- U4 pad 4: RGB4 -> (no net)
- U4 pad 5: RGB5 -> (no net)
- U40 pad 1: Net-(D40-Pad2) -> COL7
- U40 pad 2: COL7 -> ROW4
- U40 pad 3: GND -> (no net)
- U40 pad 4: RGB24 -> (no net)
- U40 pad 5: RGB25 -> (no net)
- U41 pad 1: Net-(D41-Pad2) -> COL8
- U41 pad 2: COL8 -> ROW4
- U41 pad 3: GND -> (no net)
- U41 pad 4: RGB25 -> (no net)
- U41 pad 5: RGB26 -> (no net)
- U42 pad 1: Net-(D42-Pad2) -> COL9
- U42 pad 2: COL9 -> ROW4
- U42 pad 3: GND -> (no net)
- U42 pad 4: RGB26 -> (no net)
- U42 pad 5: RGB27 -> (no net)
- U43 pad 1: Net-(D43-Pad2) -> COL10
- U43 pad 2: COL10 -> ROW4
- U43 pad 3: GND -> (no net)
- U43 pad 4: RGB27 -> (no net)
- U43 pad 5: RGB28 -> (no net)
- U44 pad 1: Net-(D44-Pad2) -> COL11
- U44 pad 2: COL11 -> ROW4
- U44 pad 3: GND -> (no net)
- U44 pad 4: RGB28 -> (no net)
- U44 pad 5: RGB29 -> (no net)
- U45 pad 1: /RP2040/QSPISS -> /Sheet61BBB357/P1.11
- U45 pad 2: /RP2040/SQPISD1 -> BLUE_LED
- U45 pad 3: /RP2040/QSPISD2 -> COL4
- U45 pad 4: GND -> COL3
- U45 pad 5: /RP2040/QSPISD0 -> GND
- U45 pad 6: /RP2040/QSPICLK -> ROW4
- U45 pad 7: /RP2040/QSPISD3 -> ROW3
- U45 pad 8: +3V3 -> ROW2
- U46 pad 1: +3V3 -> Net-(R5-Pad2)
- U46 pad 2: COL1 -> GND
- U46 pad 3: COL2 -> VBAT
- U46 pad 4: COL3 -> VBUS
- U46 pad 5: COL4 -> Net-(R6-Pad2)
- U5 pad 1: Net-(D5-Pad2) -> COL5
- U5 pad 2: COL5 -> ROW1
- U5 pad 3: GND -> (no net)
- U5 pad 4: RGB5 -> (no net)
- U5 pad 5: RGB6 -> (no net)
- U6 pad 1: Net-(D6-Pad2) -> COL6
- U6 pad 2: COL6 -> ROW1
- U6 pad 3: GND -> (no net)
- U6 pad 4: RGB16 -> (no net)
- U6 pad 5: RGB17 -> (no net)
- U7 pad 1: Net-(D7-Pad2) -> COL7
- U7 pad 2: COL7 -> ROW1
- U7 pad 3: GND -> (no net)
- U7 pad 4: RGB40 -> (no net)
- U7 pad 5: RGB41 -> (no net)
- U8 pad 1: Net-(D8-Pad2) -> COL8
- U8 pad 2: COL8 -> ROW1
- U8 pad 3: GND -> (no net)
- U8 pad 4: RGB41 -> (no net)
- U8 pad 5: RGB42 -> (no net)
- U9 pad 1: Net-(D9-Pad2) -> COL9
- U9 pad 2: COL9 -> ROW1
- U9 pad 3: GND -> (no net)
- U9 pad 4: RGB42 -> (no net)
- U9 pad 5: RGB43 -> (no net)
- Y1 pad 1: /RP2040/XIN -> Net-(C1-Pad1)
- Y1 pad 2: GND -> Net-(C2-Pad2)
Routing:
- net +3V3: track 1487.9 -> 28.5 mm, vias 4 -> 3
- net RGB11: track 122.7 -> 0.00 mm, vias 4 -> 0
- net RGB17: track 110.4 -> 0.00 mm, vias 4 -> 0
- net RGB6: track 109.5 -> 0.00 mm
- net RGB29: track 107.1 -> 0.00 mm, vias 4 -> 0
- net RGBData1: track 106.0 -> 0.00 mm, vias 2 -> 0
- net RGB40: track 98.2 -> 0.00 mm, vias 2 -> 0
- net RGB35: track 85.2 -> 0.00 mm, vias 2 -> 0
- net COL10: track 131.8 -> 189.9 mm, vias 2 -> 1
- net LED: track 57.1 -> 0.00 mm, vias 2 -> 0
- net VBAT: track 0.00 -> 54.3 mm, vias 0 -> 2
- net RED_LED: track 0.00 -> 52.8 mm, vias 0 -> 2
- net BLUE_LED: track 0.00 -> 51.6 mm, vias 0 -> 2
- net COL11: track 152.7 -> 202.3 mm, vias 2 -> 1
- net /RP2040/RESET: track 48.8 -> 0.00 mm
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- removed copper zone on B.Cu, net +3V3
- removed copper zone on B.Cu, net GND
- removed copper zone on F.Cu, net GND
Other:
- board size 234 x 88 mm -> 232.1 x 86.2 mm
- board text added: "License: CERN-OHL-W https://github.com/jpconstantineau/VColPG1232-44 By JPConstantineau 2021-11-02"
- board text added: "ON OFF"
- board text added: "VBatt GND"
- board text added: "VColPG1232-44"
- board text added: "Vcc GND CLK SWDIO"
- board text removed: "Boot Run"
- board text removed: "JLCJLCJLCJLC"
- board text removed: "License: CERN-OHL-W https://github.com/jpconstantineau/VColChoc44 By JPConstantineau 2021-10-03"
- board text removed: "VColChoc44"
