File: VColChoc44.sch (KiCad schematic (older format))
At the start: 89 parts, among them U1 CherryMX_LTST-A683CEGBW-Rotat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, U10 CherryMX_LTST-A683CEGBW-Rotat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, U11 CherryMX_LTST-A683CEGBW-Rotat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, U12 CherryMX_LTST-A683CEGBW-Rotat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, U13 CherryMX_LTST-A683CEGBW-Rotat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, U14 CherryMX_LTST-A683CEGBW-Rotat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, U15 CherryMX_LTST-A683CEGBW-Rotat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, U16 CherryMX_LTST-A683CEGBW-Rotat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, U17 CherryMX_LTST-A683CEGBW-Rotat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, U18 CherryMX_LTST-A683CEGBW-Rotat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, U19 CherryMX_LTST-A683CEGBW-Rotat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, U2 CherryMX_LTST-A683CEGBW-Rotat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, U20 CherryMX_LTST-A683CEGBW-Rotat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, U21 CherryMX_LTST-A683CEGBW-Rotat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, U22 CherryMX_LTST-A683CEGBW-Rotat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, U23 CherryMX_LTST-A683CEGBW-Rotat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, U24 CherryMX_LTST-A683CEGBW-Rotat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, U25 CherryMX_LTST-A683CEGBW-Rotat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, U26 CherryMX_LTST-A683CEGBW-Rotat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, U27 CherryMX_LTST-A683CEGBW-Rotat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, U28 CherryMX_LTST-A683CEGBW-Rotat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, U29 CherryMX_LTST-A683CEGBW-Rotat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, U3 CherryMX_LTST-A683CEGBW-Rotat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, U30 CherryMX_LTST-A683CEGBW-Rotat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, U31 CherryMX_LTST-A683CEGBW-Rotat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, U32 CherryMX_LTST-A683CEGBW-Rotat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, U33 CherryMX_LTST-A683CEGBW-Rotat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, U34 CherryMX_LTST-A683CEGBW-Rotat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, U35 CherryMX_LTST-A683CEGBW-Rotat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, U36 CherryMX_LTST-A683CEGBW-Rotat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, U37 CherryMX_LTST-A683CEGBW-Rotat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, U38 CherryMX_LTST-A683CEGBW-Rotat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, U39 CherryMX_LTST-A683CEGBW-Rotat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, U4 CherryMX_LTST-A683CEGBW-Rotat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, U40 CherryMX_LTST-A683CEGBW-Rotat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, U41 CherryMX_LTST-A683CEGBW-Rotat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, U42 CherryMX_LTST-A683CEGBW-Rotat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, U43 CherryMX_LTST-A683CEGBW-Rotat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, U44 CherryMX_LTST-A683CEGBW-Rotat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, U5 CherryMX_LTST-A683CEGBW-Rotat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, U6 CherryMX_LTST-A683CEGBW-Rotat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, U7 CherryMX_LTST-A683CEGBW-Rotat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, U8 CherryMX_LTST-A683CEGBW-Rotat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, U9 CherryMX_LTST-A683CEGBW-Rotat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

Commit message: initial
Parts:
- removed D1, D10, D11, D12, D13, D14, D15, D16, D17, D18, D19, D2, D20, D21, D22, D23, D24, D25, D26, D27, D28, D29, D3, D30, D31, D32, D33, D34, D35, D36, D37, D38, D39, D4, D40, D41, D42, D43, D44, D5, D6, D7, D8, D9: D, Diode_SMD:D_SOD-123, symbol Device:D
- removed U1, U10, U11, U12, U13, U14, U15, U16, U17, U18, U19, U2, U20, U21, U22, U23, U24, U25, U26, U27, U28, U29, U3, U30, U31, U32, U33, U34, U35, U36, U37, U38, U39, U4, U40, U41, U42, U43, U44, U5, U6, U7, U8, U9: CherryMX_LTST-A683CEGBW-Rotated, keyswitches:Kailh_socket_PG1350_sk6812mini_e, symbol CherryMX:CherryMX_LTST-A683CEGBW-Rotated
- added H1, H10, H2, H3, H4, H5, H6, H7, H8, H9: MountingHole, MountingHole:MountingHole_2.2mm_M2_DIN965, symbol Mechanical:MountingHole
- added U1, U10, U11, U12, U13, U14, U15, U16, U17, U18, U19, U2, U20, U21, U22, U23, U24, U25, U26, U27, U28, U29, U3, U30, U31, U32, U33, U34, U35, U36, U37, U38, U39, U4, U40, U41, U42, U43, U44, U5, U6, U7, U8, U9: diode-choc, pg1232:pg1232-D, symbol diode-choc:diode-choc
Connections:
- net COL1: now also U1.1, U12.1, U23.1, U34.1
- net COL10: now also U10.1, U21.1, U32.1, U43.1
- net COL11: now also U11.1, U22.1, U33.1, U44.1
- net COL2: now also U13.1, U2.1, U24.1, U35.1
- net COL3: now also U14.1, U25.1, U3.1, U36.1
- net COL4: now also U15.1, U26.1, U37.1, U4.1
- net COL5: now also U16.1, U27.1, U38.1, U5.1
- net COL6: now also U17.1, U28.1, U39.1, U6.1
- net COL7: now also U18.1, U29.1, U40.1, U7.1
- net COL8: now also U19.1, U30.1, U41.1, U8.1
- net COL9: now also U20.1, U31.1, U42.1, U9.1
- net ROW1: now also U1.2, U10.2, U11.2, U2.2, U3.2, U4.2, U5.2, U6.2, U7.2, U8.2, U9.2
- net ROW2: now also U12.2, U13.2, U14.2, U15.2, U16.2, U17.2, U18.2, U19.2, U20.2, U21.2, U22.2
- net ROW3: now also U23.2, U24.2, U25.2, U26.2, U27.2, U28.2, U29.2, U30.2, U31.2, U32.2, U33.2
- net ROW4: now also U34.2, U35.2, U36.2, U37.2, U38.2, U39.2, U40.2, U41.2, U42.2, U43.2, U44.2
- no-connect marks 1 -> 0
